Commit message: updated to use livox mesh as visual

File: urdf/mid360.xacro (robot description, xacro)
@@ -1,11 +1,11 @@
 <?xml version="1.0" encoding="UTF-8"?>
 <robot xmlns:xacro="http://ros.org/wiki/xacro">
-  <xacro:property name="M_PI" value="3.1415926"/>
-  <xacro:property name="laser_min_range" value="0.1"/>
-  <xacro:property name="laser_max_range" value="200.0"/>
-  <xacro:property name="samples" value="40000"/>
-  <xacro:property name="resolution" value="0.002"/>
-  <xacro:property name="noise_mean" value="0.0"/>
-  <xacro:property name="noise_stddev" value="0.01"/>
+  <xacro:property name="M_PI" value="3.1415926" />
+  <xacro:property name="laser_min_range" value="0.1" />
+  <xacro:property name="laser_max_range" value="200.0" />
+  <xacro:property name="samples" value="40000" />
+  <xacro:property name="resolution" value="0.002" />
+  <xacro:property name="noise_mean" value="0.0" />
+  <xacro:property name="noise_stddev" value="0.01" />
   <xacro:property name="mass" value="0.4" />
   <xacro:property name="length" value="0.1" />
@@ -14,22 +14,32 @@
   <xacro:macro name="box_inertia" params="m w h d">
     <inertial>
-      <origin xyz="0 0 0" rpy="${pi/2} 0 ${pi/2}"/>
-      <mass value="${m}"/>
-      <inertia ixx="${(m/12) * (h*h + d*d)}" ixy="0.0" ixz="0.0" iyy="${(m/12) * (w*w + d*d)}" iyz="0.0" izz="${(m/12) * (w*w + h*h)}"/>
+      <origin xyz="0 0 0" rpy="${pi/2} 0 ${pi/2}" />
+      <mass value="${m}" />
+      <inertia ixx="${(m/12) * (h*h + d*d)}" ixy="0.0" ixz="0.0" iyy="${(m/12) * (w*w + d*d)}"
+        iyz="0.0" izz="${(m/12) * (w*w + h*h)}" />
     </inertial>
   </xacro:macro>
-  <xacro:macro name="mid360" params="name:='' parent:= 'base_link' topic:='mid360' *origin ">
-<link name="${name}">
-<xacro:box_inertia m="${length}" w="${width}" d="${length}" h="${height}"/>
-  <visual>
+  <xacro:macro name="mid360" params="name:='' parent:= 'base_link' yaw:='0' robot:='' topic:='mid360' *origin ">
+    <link name="${name}">
+      <xacro:box_inertia m="${length}" w="${width}" d="${length}" h="${height}" />
+      <visual>
+        <origin xyz="0 0 -0.047" rpy="0 0 ${yaw}" />
         <geometry>
-            <box size="${length} ${width} ${height}"/>
+            <mesh
+                filename="file://$(find drc_flexnav_description)/meshes/${robot}/lidar.dae" />
         </geometry>
-  </visual>
-</link>
+    </visual>
+    <collision>
+        <origin xyz="0 0 -0.047" rpy="0 0 ${yaw}" />
+        <geometry>
+            <mesh
+                filename="file://$(find drc_flexnav_description)/meshes/${robot}/lidar.dae" />
+        </geometry>
+    </collision>
+    </link>
     <joint name="${name}_joint" type="fixed">
-      <parent link="${parent}"/>
-      <child link="${name}"/>
-      <xacro:insert_block name="origin"/>
+      <parent link="${parent}" />
+      <child link="${name}" />
+      <xacro:insert_block name="origin" />
     </joint>
     <gazebo reference="${name}">
@@ -40,35 +50,35 @@
         <!-- This ray plgin is only for visualization. -->
         <plugin name="${name}_plugin" filename="libros2_livox.so">
-			<ray>
-			  <scan>
-				<horizontal>
-				<samples>100</samples>
-				<resolution>1</resolution>
-				<min_angle>${0}</min_angle>
-				<max_angle>${2*M_PI}</max_angle>
-				</horizontal>
-				<vertical>
-				<samples>360</samples>
-				<resolution>1</resolution>
-				<min_angle>${-7.22/180*M_PI}</min_angle>
-				<max_angle>${55.22/180*M_PI}</max_angle>
-				</vertical>
-			  </scan>
-			  <range>
-				<min>${laser_min_range}</min>
-				<max>${laser_max_range}</max>
-				<resolution>${resolution}</resolution>
-			  </range>
-			  <noise>
-				<type>gaussian</type>
-				<mean>${noise_mean}</mean>
-				<stddev>${noise_stddev}</stddev>
-			  </noise>
-			</ray>
+          <ray>
+            <scan>
+              <horizontal>
+                <samples>100</samples>
+                <resolution>1</resolution>
+                <min_angle>${0}</min_angle>
+                <max_angle>${2*M_PI}</max_angle>
+              </horizontal>
+              <vertical>
+                <samples>360</samples>
+                <resolution>1</resolution>
+                <min_angle>${-7.22/180*M_PI}</min_angle>
+                <max_angle>${55.22/180*M_PI}</max_angle>
+              </vertical>
+            </scan>
+            <range>
+              <min>${laser_min_range}</min>
+              <max>${laser_max_range}</max>
+              <resolution>${resolution}</resolution>
+            </range>
+            <noise>
+              <type>gaussian</type>
+              <mean>${noise_mean}</mean>
+              <stddev>${noise_stddev}</stddev>
+            </noise>
+          </ray>
           <visualize>false</visualize>
-		  <samples>${samples}</samples>
-		  <downsample>1</downsample>
-		  <csv_file_name>$(find ros2_livox_simulation)/scan_mode/mid360.csv</csv_file_name>
-		  <topic>${topic}</topic>
+          <samples>${samples}</samples>
+          <downsample>1</downsample>
+          <csv_file_name>$(find ros2_livox_simulation)/scan_mode/mid360.csv</csv_file_name>
+          <topic>${topic}</topic>
         </plugin>
       </sensor>

Commit message: fix: ray distance measurement and lidar visual

File: urdf/mid360.xacro (robot description, xacro)
@@ -22,9 +22,4 @@
 <link name="${name}">
 <xacro:box_inertia m="${length}" w="${width}" d="${length}" h="${height}"/>
-  <visual>
-        <geometry>
-            <box size="${length} ${width} ${height}"/>
-        </geometry>
-  </visual>
 </link>
     <joint name="${name}_joint" type="fixed">

Commit message: fix: updates samples value to 20k

File: urdf/mid360.xacro (robot description, xacro)
@@ -4,5 +4,5 @@
   <xacro:property name="laser_min_range" value="0.1"/>
   <xacro:property name="laser_max_range" value="200.0"/>
-  <xacro:property name="samples" value="40000"/>
+  <xacro:property name="samples" value="20000"/>
   <xacro:property name="resolution" value="0.002"/>
   <xacro:property name="noise_mean" value="0.0"/>

Commit message: added livox mesh to urdf

File: urdf/mid360.xacro (robot description, xacro)
@@ -19,8 +19,20 @@
     </inertial>
   </xacro:macro>
-  <xacro:macro name="mid360" params="name:='' parent:= 'base_link' topic:='mid360' *origin ">
-<link name="${name}">
-<xacro:box_inertia m="${length}" w="${width}" d="${length}" h="${height}"/>
-</link>
+  <xacro:macro name="mid360" params="name:='' parent:= 'base_link' topic:='mid360' robot:='flexnav1500' *origin  ">
+    <link name="${name}">
+      <xacro:box_inertia m="${length}" w="${width}" d="${length}" h="${height}"/>
+      <visual>
+        <origin xyz="0 0 0" rpy="0 0 0" />
+        <geometry>
+          <mesh filename="file://$(find drc_flexnav_description)/meshes/${robot}/lidar.dae" />
+        </geometry>
+      </visual>
+      <collision>
+        <origin xyz="0 0 0" rpy="0 0 0" />
+        <geometry>
+          <mesh filename="file://$(find drc_flexnav_description)/meshes/${robot}/lidar.dae" />
+        </geometry>
+      </collision>
+    </link>
     <joint name="${name}_joint" type="fixed">
       <parent link="${parent}"/>
@@ -35,35 +47,35 @@
         <!-- This ray plgin is only for visualization. -->
         <plugin name="${name}_plugin" filename="libros2_livox.so">
-			<ray>
-			  <scan>
-				<horizontal>
-				<samples>100</samples>
-				<resolution>1</resolution>
-				<min_angle>${0}</min_angle>
-				<max_angle>${2*M_PI}</max_angle>
-				</horizontal>
-				<vertical>
-				<samples>360</samples>
-				<resolution>1</resolution>
-				<min_angle>${-7.22/180*M_PI}</min_angle>
-				<max_angle>${55.22/180*M_PI}</max_angle>
-				</vertical>
-			  </scan>
-			  <range>
-				<min>${laser_min_range}</min>
-				<max>${laser_max_range}</max>
-				<resolution>${resolution}</resolution>
-			  </range>
-			  <noise>
-				<type>gaussian</type>
-				<mean>${noise_mean}</mean>
-				<stddev>${noise_stddev}</stddev>
-			  </noise>
-			</ray>
+          <ray>
+            <scan>
+              <horizontal>
+                <samples>100</samples>
+                <resolution>1</resolution>
+                <min_angle>${0}</min_angle>
+                <max_angle>${2*M_PI}</max_angle>
+              </horizontal>
+              <vertical>
+                <samples>360</samples>
+                <resolution>1</resolution>
+                <min_angle>${-7.22/180*M_PI}</min_angle>
+                <max_angle>${55.22/180*M_PI}</max_angle>
+              </vertical>
+            </scan>
+            <range>
+              <min>${laser_min_range}</min>
+              <max>${laser_max_range}</max>
+              <resolution>${resolution}</resolution>
+            </range>
+            <noise>
+              <type>gaussian</type>
+              <mean>${noise_mean}</mean>
+              <stddev>${noise_stddev}</stddev>
+            </noise>
+          </ray>
           <visualize>false</visualize>
-		  <samples>${samples}</samples>
-		  <downsample>1</downsample>
-		  <csv_file_name>$(find ros2_livox_simulation)/scan_mode/mid360.csv</csv_file_name>
-		  <topic>${topic}</topic>
+          <samples>${samples}</samples>
+          <downsample>1</downsample>
+          <csv_file_name>$(find ros2_livox_simulation)/scan_mode/mid360.csv</csv_file_name>
+          <topic>${topic}</topic>
         </plugin>
       </sensor>

Commit message: remove drc dependencies, add mid360 meshe

File: urdf/mid360.xacro (robot description, xacro)
@@ -26,5 +26,5 @@
         <origin xyz="0 0 -0.047" rpy="0 0 0" />
         <geometry>
-          <mesh filename="file://$(find drc_flexnav_description)/meshes/${robot}/lidar.dae" />
+          <mesh filename="file://$(find ros2_livox_simulation)/meshes/mid360.dae" />
         </geometry>
       </visual>
@@ -32,5 +32,5 @@
         <origin xyz="0 0 -0.047" rpy="0 0 0" />
         <geometry>
-          <mesh filename="file://$(find drc_flexnav_description)/meshes/${robot}/lidar.dae" />
+          <mesh filename="file://$(find ros2_livox_simulation)/meshes/mid360.dae" />
         </geometry>
       </collision>

Commit message: feat: vertical and horizontal angle limits as input parameters

File: urdf/mid360.xacro (robot description, xacro)
@@ -4,4 +4,8 @@
   <xacro:property name="laser_min_range" value="0.1"/>
   <xacro:property name="laser_max_range" value="200.0"/>
+  <xacro:property name="horizontal_min_angle" value="${-M_PI}"/>
+  <xacro:property name="horizontal_max_angle" value="${M_PI}"/>
+  <xacro:property name="vertical_min_angle" value="${-M_PI/2}"/>
+  <xacro:property name="vertical_max_angle" value="${M_PI/2}"/>
   <xacro:property name="samples" value="20000"/>
   <xacro:property name="resolution" value="0.002"/>
@@ -53,12 +57,12 @@
                 <samples>100</samples>
                 <resolution>1</resolution>
-                <min_angle>${-M_PI}</min_angle>
-                <max_angle>${M_PI}</max_angle>
+                <min_angle>${horizontal_min_angle}</min_angle>
+                <max_angle>${horizontal_max_angle}</max_angle>
               </horizontal>
               <vertical>
                 <samples>360</samples>
                 <resolution>1</resolution>
-                <min_angle>${-M_PI/2}</min_angle>
-                <max_angle>${M_PI/2}</max_angle>
+                <min_angle>${vertical_min_angle}</min_angle>
+                <max_angle>${vertical_max_angle}</max_angle>
               </vertical>
             </scan>
